Commit message: Working with collision and inertia of the agribot

File: agribot_description/urdf/mech/base_mesh.urdf.xacro (robot description, xacro)
@@ -1,13 +1,34 @@
 <?xml version="1.0"?>
 <robot xmlns:xacro="http://ros.org/wiki/xacro">
-  <xacro:macro name="base_mesh" params="mesh_file">
+<xacro:macro name="base_mesh" params="
+      mesh_file
+      mass com
+      ixx iyy izz ixy ixz iyz">
     <link name="base_footprint"/>
     <link name="base_link">
+      <inertial>
+        <origin xyz="${com}" rpy="0 0 0"/>
+        <mass value="${mass}"/>
+        <inertia
+          ixx="${ixx}" iyy="${iyy}" izz="${izz}"
+          ixy="${ixy}" ixz="${ixz}" iyz="${iyz}"/>
+      </inertial>
       <visual>
-        <origin xyz="0 0 0" rpy="0 0 0"/>
         <geometry>
           <mesh filename="${mesh_file}" scale="0.001 0.001 0.001"/>
         </geometry>
       </visual>
+      <collision>
+        <origin xyz="0 0 0" rpy="0 0 0"/>
+        <geometry>
+          <box size="0.18986 0.3838 0.0269" />
+        </geometry>
+      </collision>
+      <collision>
+        <origin xyz="0.09493 0.1919 -0.18" rpy="0 2.355 0"/>
+        <geometry>
+          <cylinder length="0.33118" radius="0.0119" />
+        </geometry>
+      </collision>
     </link>
     <joint name="base_joint" type="fixed">

File: agribot_description/urdf/mech/wheel_mesh.urdf.xacro (robot description, xacro)
@@ -1,6 +1,16 @@
 <?xml version="1.0"?>
 <robot xmlns:xacro="http://ros.org/wiki/xacro">
-  <xacro:macro name="wheel_mesh" params="mesh_file parent joint_name link_name xyz rpy axis">
+  <xacro:macro name="wheel_mesh" params="
+      mesh_file parent joint_name link_name xyz rpy axis
+      mass com
+      ixx iyy izz ixy ixz iyz">
     <link name="${link_name}">
+      <inertial>
+        <origin xyz="${com}" rpy="0 0 0"/>
+        <mass value="${mass}"/>
+        <inertia
+          ixx="${ixx}" iyy="${iyy}" izz="${izz}"
+          ixy="${ixy}" ixz="${ixz}" iyz="${iyz}"/>
+      </inertial>
       <visual>
         <origin xyz="0 0 0" rpy="0 0 0"/>
@@ -9,4 +19,10 @@
         </geometry>
       </visual>
+      <collision>
+        <origin xyz="0 0 0" rpy="0 0 0"/>
+        <geometry>
+          <mesh filename="${mesh_file}" scale="0.001 0.001 0.001"/>
+        </geometry>
+      </collision>
     </link>
     <joint name="${joint_name}" type="continuous">

File: agribot_description/urdf/properties/agribot.properties.xacro (robot description, xacro)
@@ -19,5 +19,23 @@
   <xacro:property name="wheel_axis" value="0 1 0"/>
   <!-- For later: controllers/odom math (placeholder until measured) -->
-  <xacro:property name="wheel_separation" value="0.45946"/> <!-- 2*0.22973 -->
-  <xacro:property name="wheel_radius" value="0.10"/> <!-- TODO: set real radius in meters -->
+  <xacro:property name="wheel_separation" value="0.51"/>
+  <xacro:property name="wheel_radius" value="0.05"/>
+    <!-- Base inertial (Fusion -> URDF SI units) -->
+  <xacro:property name="base_mass" value="4.248128"/>
+  <xacro:property name="base_com"  value="0.02623 -0.000536 -0.042696"/>
+  <xacro:property name="base_ixx" value="0.1076"/>
+  <xacro:property name="base_iyy" value="0.1189"/>
+  <xacro:property name="base_izz" value="0.1484"/>
+  <xacro:property name="base_ixy" value="0.000001115543"/>
+  <xacro:property name="base_ixz" value="-0.003339"/>
+  <xacro:property name="base_iyz" value="0.0002084"/>
+  <!-- Wheel inertial -->
+  <xacro:property name="wheel_mass" value="0.223669"/>
+  <xacro:property name="wheel_com"  value="0 0.001512 0"/>
+  <xacro:property name="wheel_ixx" value="0.000183"/>
+  <xacro:property name="wheel_iyy" value="0.0003286"/>
+  <xacro:property name="wheel_izz" value="0.000183"/>
+  <xacro:property name="wheel_ixy" value="0.0"/>
+  <xacro:property name="wheel_ixz" value="0.0"/>
+  <xacro:property name="wheel_iyz" value="0.0"/>
 </robot>

File: agribot_description/urdf/robots/agribot.urdf.xacro (robot description, xacro)
@@ -7,24 +7,47 @@
   <xacro:include filename="$(find agribot_description)/urdf/mech/wheel_mesh.urdf.xacro"/>
   <!-- Base -->
-  <xacro:base_mesh mesh_file="${base_mesh_file}"/>
+    <xacro:base_mesh
+    mesh_file="${base_mesh_file}"
+    mass="${base_mass}"
+    com="${base_com}"
+    ixx="${base_ixx}" iyy="${base_iyy}" izz="${base_izz}"
+    ixy="${base_ixy}" ixz="${base_ixz}" iyz="${base_iyz}"/>
   <!-- Left wheels -->
   <xacro:wheel_mesh mesh_file="${left_wheel_mesh_file}" parent="base_link"
     joint_name="left_wheel_front_joint" link_name="left_wheel_link_front"
-    xyz="${lf_xyz}" rpy="${wheel_rpy}" axis="${wheel_axis}"/>
+    xyz="${lf_xyz}" rpy="${wheel_rpy}" axis="${wheel_axis}"
+    mass="${wheel_mass}" com="${wheel_com}"
+    ixx="${wheel_ixx}" iyy="${wheel_iyy}" izz="${wheel_izz}"
+    ixy="${wheel_ixy}" ixz="${wheel_ixz}" iyz="${wheel_iyz}"/>
   <xacro:wheel_mesh mesh_file="${left_wheel_mesh_file}" parent="base_link"
     joint_name="left_wheel_mid_joint" link_name="left_wheel_link_mid"
-    xyz="${lm_xyz}" rpy="${wheel_rpy}" axis="${wheel_axis}"/>
+    xyz="${lm_xyz}" rpy="${wheel_rpy}" axis="${wheel_axis}"
+    mass="${wheel_mass}" com="${wheel_com}"
+    ixx="${wheel_ixx}" iyy="${wheel_iyy}" izz="${wheel_izz}"
+    ixy="${wheel_ixy}" ixz="${wheel_ixz}" iyz="${wheel_iyz}"/>
   <xacro:wheel_mesh mesh_file="${left_wheel_mesh_file}" parent="base_link"
     joint_name="left_wheel_rear_joint" link_name="left_wheel_link_rear"
-    xyz="${lr_xyz}" rpy="${wheel_rpy}" axis="${wheel_axis}"/>
+    xyz="${lr_xyz}" rpy="${wheel_rpy}" axis="${wheel_axis}"
+    mass="${wheel_mass}" com="${wheel_com}"
+    ixx="${wheel_ixx}" iyy="${wheel_iyy}" izz="${wheel_izz}"
+    ixy="${wheel_ixy}" ixz="${wheel_ixz}" iyz="${wheel_iyz}"/>
   <!-- Right wheels -->
   <xacro:wheel_mesh mesh_file="${right_wheel_mesh_file}" parent="base_link"
     joint_name="right_wheel_front_joint" link_name="right_wheel_link_front"
-    xyz="${rf_xyz}" rpy="${wheel_rpy}" axis="${wheel_axis}"/>
+    xyz="${rf_xyz}" rpy="${wheel_rpy}" axis="${wheel_axis}"
+    mass="${wheel_mass}" com="${wheel_com}"
+    ixx="${wheel_ixx}" iyy="${wheel_iyy}" izz="${wheel_izz}"
+    ixy="${wheel_ixy}" ixz="${wheel_ixz}" iyz="${wheel_iyz}"/>
   <xacro:wheel_mesh mesh_file="${right_wheel_mesh_file}" parent="base_link"
     joint_name="right_wheel_mid_joint" link_name="right_wheel_link_mid"
-    xyz="${rm_xyz}" rpy="${wheel_rpy}" axis="${wheel_axis}"/>
+    xyz="${rm_xyz}" rpy="${wheel_rpy}" axis="${wheel_axis}"
+    mass="${wheel_mass}" com="${wheel_com}"
+    ixx="${wheel_ixx}" iyy="${wheel_iyy}" izz="${wheel_izz}"
+    ixy="${wheel_ixy}" ixz="${wheel_ixz}" iyz="${wheel_iyz}"/>
   <xacro:wheel_mesh mesh_file="${right_wheel_mesh_file}" parent="base_link"
     joint_name="right_wheel_rear_joint" link_name="right_wheel_link_rear"
-    xyz="${rr_xyz}" rpy="${wheel_rpy}" axis="${wheel_axis}"/>
+    xyz="${rr_xyz}" rpy="${wheel_rpy}" axis="${wheel_axis}"
+    mass="${wheel_mass}" com="${wheel_com}"
+    ixx="${wheel_ixx}" iyy="${wheel_iyy}" izz="${wheel_izz}"
+    ixy="${wheel_ixy}" ixz="${wheel_ixz}" iyz="${wheel_iyz}"/>
 </robot>

Commit message: Done with collision now moving to ros2_control i.e differential drive now .

File: agribot_description/urdf/mech/base_mesh.urdf.xacro (robot description, xacro)
@@ -19,14 +19,61 @@
         </geometry>
       </visual>
+      <!--Collision for box of base link-->
       <collision>
         <origin xyz="0 0 0" rpy="0 0 0"/>
         <geometry>
-          <box size="0.18986 0.3838 0.0269" />
+          <box size="0.19986 0.4238 0.0269" />
+        </geometry>
+      </collision>
+      <!--Collision for rocker left side-->
+      <collision>
+        <origin xyz="0.21986 0.2038 -0.12059" rpy="0 2.255 0"/>
+        <geometry>
+          <cylinder length="0.3568" radius="0.0119" />
+        </geometry>
+      </collision>
+      <!--Collision for rocker right side-->
+      <collision>
+        <origin xyz="0.21986 -0.2038 -0.12059" rpy="0 2.255 0"/>
+        <geometry>
+          <cylinder length="0.3568" radius="0.0119" />
+        </geometry>
+      </collision>
+      <!--Collision for bogie left side-->
+      <collision>
+        <origin xyz="-0.12493 0.2038 -0.042465" rpy="0 0.785 0"/>
+        <geometry>
+          <cylinder length="0.10493" radius="0.0119" />
         </geometry>
       </collision>
       <collision>
-        <origin xyz="0.09493 0.1919 -0.18" rpy="0 2.355 0"/>
+        <origin xyz="-0.246395 0.2038 -0.16393" rpy="0 0.785 0"/>
         <geometry>
-          <cylinder length="0.33118" radius="0.0119" />
+          <cylinder length="0.24293" radius="0.0119" />
+        </geometry>
+      </collision>
+      <collision>
+        <origin xyz="-0.086395 0.2038 -0.16393" rpy="0 2.255 0"/>
+        <geometry>
+          <cylinder length="0.24293" radius="0.0119" />
+        </geometry>
+      </collision>
+      <!--Collision for bogie right side-->
+      <collision>
+        <origin xyz="-0.12493 -0.2038 -0.042465" rpy="0 0.785 0"/>
+        <geometry>
+          <cylinder length="0.10493" radius="0.0119" />
+        </geometry>
+      </collision>
+      <collision>
+        <origin xyz="-0.246395 -0.2038 -0.16393" rpy="0 0.785 0"/>
+        <geometry>
+          <cylinder length="0.24293" radius="0.0119" />
+        </geometry>
+      </collision>
+      <collision>
+        <origin xyz="-0.086395 -0.2038 -0.16393" rpy="0 2.255 0"/>
+        <geometry>
+          <cylinder length="0.24293" radius="0.0119" />
         </geometry>
       </collision>

File: agribot_description/urdf/mech/wheel_mesh.urdf.xacro (robot description, xacro)
@@ -20,7 +20,7 @@
       </visual>
       <collision>
-        <origin xyz="0 0 0" rpy="0 0 0"/>
+        <origin xyz="0 0 0" rpy="1.57 0 0"/>
         <geometry>
-          <mesh filename="${mesh_file}" scale="0.001 0.001 0.001"/>
+          <cylinder length="0.045" radius="0.052" />
         </geometry>
       </collision>
