Commit message: Differential drive controller is wokring now. With ros2_controller for gazebodone. Now manual teleoperation of bot is sucessful. Now we will move to adding sensors like imu, doing ekf and then adding lidar after getting stable odom.

File: agribot_description/urdf/properties/agribot.properties.xacro (robot description, xacro)
@@ -1,11 +1,11 @@
 <?xml version="1.0"?>
 <robot xmlns:xacro="http://ros.org/wiki/xacro">
-  <!-- Meshes -->
+  <xacro:property name="pkg_share" value="$(find agribot_description)"/>
   <xacro:property name="base_mesh_file"
-    value="package://agribot_description/meshes/agribot_baselink.stl"/>
+    value="file://${pkg_share}/meshes/agribot_baselink.stl"/>
   <xacro:property name="left_wheel_mesh_file"
-    value="package://agribot_description/meshes/agribot_left_wheel.stl"/>
+    value="file://${pkg_share}/meshes/agribot_left_wheel.stl"/>
   <xacro:property name="right_wheel_mesh_file"
-    value="package://agribot_description/meshes/agribot_right_wheel.stl"/>
+    value="file://${pkg_share}/meshes/agribot_right_wheel.stl"/>
   <!-- Wheel joint origins (copied from your URDF) -->
   <xacro:property name="lf_xyz" value="0.35606  0.22973 -0.22532" />

File: agribot_description/urdf/robots/agribot.urdf.xacro (robot description, xacro)
@@ -3,4 +3,7 @@
   <!-- Properties -->
   <xacro:include filename="$(find agribot_description)/urdf/properties/agribot.properties.xacro"/>
+  <!--Gazebo and ros2 control plugins-->
+  <xacro:include filename="$(find agribot_description)/urdf/control/agribot.ros2control.xacro"/>
+  <xacro:include filename="$(find agribot_description)/urdf/control/agribot.gazebo.xacro"/>
   <!-- Mech -->
   <xacro:include filename="$(find agribot_description)/urdf/mech/base_mesh.urdf.xacro"/>

Commit message: updated for ekf Differential drive controller with manual teleoperation is working .

File: agribot_description/urdf/properties/agribot.properties.xacro (robot description, xacro)
@@ -20,5 +20,5 @@
   <!-- For later: controllers/odom math (placeholder until measured) -->
   <xacro:property name="wheel_separation" value="0.51"/>
-  <xacro:property name="wheel_radius" value="0.05"/>
+  <xacro:property name="wheel_radius" value="0.052"/>
     <!-- Base inertial (Fusion -> URDF SI units) -->
   <xacro:property name="base_mass" value="4.248128"/>
